File: PCB/Piezo_Energy_Harvester.kicad_sch (KiCad schematic)
At the start: 9 parts, among them J1 Conn_01x01_Pin, J2 Conn_01x01_Pin, U1 LTC3588IMSE-1-PBF

Commit message: change of footprint
Parts:
- renumbered C3 to C1, C5 to C3, C1 to C4, C4 to C5
Changed lines of the file:
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@@
 		(on_board yes)
 		(dnp no)
-		(property "Reference" "C5"
+		(property "Reference" "C3"
 			(at 72.644 96.774 0)
 			(effects
@@
 			(project "Piezo_Energy_Harvester"
 				(path "/2025adb1-c4aa-48e7-bd62-33e2593b3a69"
-					(reference "C5")
+					(reference "C3")
 					(unit 1)
 				)
@@
 		(dnp no)
 		(fields_autoplaced yes)
-		(property "Reference" "#PWR01"
+		(property "Reference" "#PWR05"
 			(at 158.75 124.46 0)
 			(effects
@@
 			(project ""
 				(path "/2025adb1-c4aa-48e7-bd62-33e2593b3a69"
-					(reference "#PWR01")
+					(reference "#PWR05")
 					(unit 1)
 				)
@@
 		(on_board yes)
 		(dnp no)
-		(property "Reference" "C4"
+		(property "Reference" "C5"
 			(at 169.164 109.22 0)
 			(effects
@@
 			)
 		)
-		(property "Datasheet" "~"
+		(property "Datasheet" "https://www.mouser.pl/ProductDetail/Maxwell-Technologies/BMOD0001-P005-B02?qs=W0yvOO0ixfEzFv8%2F5TnOWA%3D%3D"
 			(at 173.99 111.76 0)
 			(effects
@@
 			(project "Piezo_Energy_Harvester"
 				(path "/2025adb1-c4aa-48e7-bd62-33e2593b3a69"
-					(reference "C4")
+					(reference "C5")
 					(unit 1)
 				)
@@
 		(dnp no)
 		(fields_autoplaced yes)
-		(property "Reference" "#PWR04"
+		(property "Reference" "#PWR01"
 			(at 179.07 90.17 0)
 			(effects
@@
 			(project "Piezo_Energy_Harvester"
 				(path "/2025adb1-c4aa-48e7-bd62-33e2593b3a69"
-					(reference "#PWR04")
+					(reference "#PWR01")
 					(unit 1)
 				)
@@
 		(dnp no)
 		(fields_autoplaced yes)
-		(property "Reference" "#PWR02"
+		(property "Reference" "#PWR04"
 			(at 175.26 104.14 0)
 			(effects
@@
 			(project ""
 				(path "/2025adb1-c4aa-48e7-bd62-33e2593b3a69"
-					(reference "#PWR02")
+					(reference "#PWR04")
 					(unit 1)
 				)
@@
 		(dnp no)
 		(fields_autoplaced yes)
-		(property "Reference" "#PWR03"
+		(property "Reference" "#PWR02"
 			(at 171.45 100.33 0)
 			(effects
@@
 			(project "Piezo_Energy_Harvester"
 				(path "/2025adb1-c4aa-48e7-bd62-33e2593b3a69"
-					(reference "#PWR03")
+					(reference "#PWR02")
 					(unit 1)
 				)
@@
 		(on_board yes)
 		(dnp no)
-		(property "Reference" "C3"
+		(property "Reference" "C1"
 			(at 71.12 85.09 0)
 			(effects
@@
 			(project "Piezo_Energy_Harvester"
 				(path "/2025adb1-c4aa-48e7-bd62-33e2593b3a69"
-					(reference "C3")
+					(reference "C1")
 					(unit 1)
 				)
@@
 		(on_board yes)
 		(dnp no)
-		(property "Reference" "C1"
+		(property "Reference" "C4"
 			(at 156.464 109.474 0)
 			(effects
@@
 			(project "Piezo_Energy_Harvester"
 				(path "/2025adb1-c4aa-48e7-bd62-33e2593b3a69"
-					(reference "C1")
+					(reference "C4")
 					(unit 1)
 				)
@@
 		(dnp no)
 		(fields_autoplaced yes)
-		(property "Reference" "#PWR05"
+		(property "Reference" "#PWR03"
 			(at 74.93 110.49 0)
 			(effects
@@
 			(project "Piezo_Energy_Harvester"
 				(path "/2025adb1-c4aa-48e7-bd62-33e2593b3a69"
-					(reference "#PWR05")
-					(unit 1)
-				)
+					(reference "#PWR03")
+					(unit 1)
+				)

Commit message: changed coil footprint
Parts:
- L1: footprint Inductor_SMD:L_0805_2012Metric_Pad1.05x1.20mm_HandSolder -> Piezo_EH_footprints:WE-HEPC_5030
Changed lines of the file:
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@@
 			)
 		)
-		(property "Footprint" "Inductor_SMD:L_0805_2012Metric_Pad1.05x1.20mm_HandSolder"
+		(property "Footprint" "Piezo_EH_footprints:WE-HEPC_5030"
 			(at 124.46 104.14 0)
 			(effects

Commit message: C4 changed
Parts:
- C4: footprint Capacitor_SMD:C_0603_1608Metric_Pad1.08x0.95mm_HandSolder -> Capacitor_SMD:CP_Elec_5x5.4
Changed lines of the file:
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@@
 			)
 		)
-		(property "Footprint" "Capacitor_SMD:C_0603_1608Metric_Pad1.08x0.95mm_HandSolder"
+		(property "Footprint" "Capacitor_SMD:CP_Elec_5x5.4"
 			(at 157.7848 107.95 0)
 			(effects

Commit message: Minor changes
Parts:
- removed C4: 47u 6V, Capacitor_SMD:CP_Elec_5x5.4, symbol Device:C
- added C4: 47u 6V, Capacitor_SMD:CP_Elec_5x5.4, symbol Device:C_Polarized
Connections:
- net +3.3V: now also C4.1
- net GND: now also C4.2
Changed lines of the file:
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@@
+	(symbol
+		(lib_id "Connector:Conn_01x01_Pin")
+		(at 73.66 80.01 0)
+		(unit 1)
+		(exclude_from_sim no)
+		(in_bom yes)
+		(on_board yes)
+		(dnp no)
+		(property "Reference" "J2"
+			(at 73.914 78.994 0)
+			(effects
+				(font
+					(size 1.27 1.27)
+				)
+			)
+		)
+		(property "Value" "Conn_01x01_Pin"
+			(at 65.278 80.01 0)
+			(effects
+				(font
+					(size 1.27 1.27)
+				)
+			)
+		)
+		(property "Footprint" "TestPoint:TestPoint_Pad_1.0x1.0mm"
+			(at 73.66 80.01 0)
+			(effects
+				(font
+					(size 1.27 1.27)
+				)
+				(hide yes)
+			)
+		)
+		(property "Datasheet" "~"
+			(at 73.66 80.01 0)
+			(effects
+				(font
+					(size 1.27 1.27)
+				)
+				(hide yes)
+			)
+		)
+		(property "Description" "Generic connector, single row, 01x01, script generated"
+			(at 73.66 80.01 0)
+			(effects
+				(font
+					(size 1.27 1.27)
+				)
+				(hide yes)
+			)
+		)
+		(pin "1"
+		)
+		(instances
+			(project "Piezo_Energy_Harvester"
+				(path "/2025adb1-c4aa-48e7-bd62-33e2593b3a69"
+					(reference "J2")
+					(unit 1)
+				)
+			)
+		)
+	)
 	(symbol
 		(lib_id "Connector:Conn_01x01_Pin")
@@
 	)
 	(symbol
-		(lib_id "Device:C")
-		(at 158.75 111.76 180)
+		(lib_id "Device:C_Polarized")
+		(at 158.75 111.76 0)
 		(unit 1)
 		(exclude_from_sim no)
@@
 		(dnp no)
 		(property "Reference" "C4"
-			(at 156.464 109.474 0)
-			(effects
-				(font
-					(size 1.27 1.27)
-				)
+			(at 153.924 109.22 0)
+			(effects
+				(font
+					(size 1.27 1.27)
+				)
+				(justify left)
 			)
 		)
 		(property "Value" "47u 6V"
-			(at 162.814 114.554 0)
-			(effects
-				(font
-					(size 1.27 1.27)
-				)
+			(at 159.512 115.316 0)
+			(effects
+				(font
+					(size 1.27 1.27)
+				)
+				(justify left)
 			)
 		)
 		(property "Footprint" "Capacitor_SMD:CP_Elec_5x5.4"
-			(at 157.7848 107.95 0)
-			(effects
-				(font
-					(size 1.27 1.27)
-				)
-				(hide yes)
-			)
-		)
-		(property "Datasheet" "~"
+			(at 159.7152 115.57 0)
+			(effects
+				(font
+					(size 1.27 1.27)
+				)
+				(hide yes)
+			)
+		)
+		(property "Datasheet" ""
 			(at 158.75 111.76 0)
 			(effects
@@
 			)
 		)
-		(property "Description" "Unpolarized capacitor"
+		(property "Description" "Polarized capacitor"
 			(at 158.75 111.76 0)
 			(effects
@@
 					(unit 1)
 				)
-			)
-		)
-	)
-	(symbol
-		(lib_id "Connector:Conn_01x01_Pin")
-		(at 73.66 80.01 0)
-		(unit 1)
-		(exclude_from_sim no)
-		(in_bom yes)
-		(on_board yes)
-		(dnp no)
-		(property "Reference" "J2"
-			(at 73.914 78.994 0)
-			(effects
-				(font
-					(size 1.27 1.27)
-				)
-			)
-		)
-		(property "Value" "Conn_01x01_Pin"
-			(at 65.278 80.01 0)
-			(effects
-				(font
-					(size 1.27 1.27)
-				)
-			)
-		)
-		(property "Footprint" "TestPoint:TestPoint_Pad_1.0x1.0mm"
-			(at 73.66 80.01 0)
-			(effects
-				(font
-					(size 1.27 1.27)
-				)
-				(hide yes)
-			)
-		)
-		(property "Datasheet" "~"
-			(at 73.66 80.01 0)
-			(effects
-				(font
-					(size 1.27 1.27)
-				)
-				(hide yes)
-			)
-		)
-		(property "Description" "Generic connector, single row, 01x01, script generated"
-			(at 73.66 80.01 0)
-			(effects
-				(font
-					(size 1.27 1.27)
-				)
-				(hide yes)
-			)
-		)
-		(pin "1"
-		)
-		(instances
-			(project "Piezo_Energy_Harvester"
-				(path "/2025adb1-c4aa-48e7-bd62-33e2593b3a69"
-					(reference "J2")
-					(unit 1)
-				)
